Commit message: Added controllers and moveit configuration

File: oscar_description/urdf/oscar.urdf.xacro (robot description, xacro)
@@ -57,45 +57,6 @@
     </collision>
   </link>
-  <!-- Call thor xacro macro
-  <link
-    name="left_arm">
-    <inertial>
-      <origin
-        xyz="0.079376 0.0040006 0.15278"
-        rpy="0 0 0" />
-      <mass
-        value="5.8547" />
-      <inertia
-        ixx="0.0070709"
-        ixy="-7.4198E-05"
-        ixz="-4.5271E-06"
-        iyy="0.011734"
-        iyz="1.6122E-06"
-        izz="0.013094" />
-    </inertial>
-    <visual>
-      <origin
-        xyz="0 0 0"
-        rpy="0 0 0" />
-      <geometry>
-        <mesh
-          filename="package://robot_description/meshes/left_arm.STL" />
-      </geometry>
-      <material
-        name="">
-        <color
-          rgba="0.75294 0.75294 0.75294 1" />
-      </material>
-    </visual>
-    <collision>
-      <origin
-        xyz="0 0 0"
-        rpy="0 0 0" />
-      <geometry>
-        <mesh
-          filename="package://robot_description/meshes/left_arm.STL" />
-      </geometry>
-    </collision>
-  </link>
+  <!-- Left arm xacro call and joint -->
+  <xacro:thor_robot prefix="left_arm_"/>
   <joint
     name="left_arm_fixed"
@@ -105,20 +66,4 @@
       rpy="0 0 0" />
     <parent
-      link="base_link" />
-    <child
-      link="left_arm" />
-    <axis
-      xyz="0 0 0" />
-  </joint>
-  -->
-  <!-- Left arm xacro call and joint -->
-  <xacro:thor_robot prefix="left_arm_"/>
-  <joint
-    name="left_arm_fixed"
-    type="fixed">
-    <origin
-      xyz="0 0.25 0.7"
-      rpy="0 0 0" />
-    <parent
       link="world" />
     <child
@@ -142,59 +87,4 @@
       xyz="0 0 0" />
   </joint>
-  <!-- Call thor xacro macro
-  <link
-    name="right_arm">
-    <inertial>
-      <origin
-        xyz="0.079376 0.0040006 0.15278"
-        rpy="0 0 0" />
-      <mass
-        value="5.8547" />
-      <inertia
-        ixx="0.0070709"
-        ixy="-7.4198E-05"
-        ixz="-4.5272E-06"
-        iyy="0.011734"
-        iyz="1.6122E-06"
-        izz="0.013094" />
-    </inertial>
-    <visual>
-      <origin
-        xyz="0 0 0"
-        rpy="0 0 0" />
-      <geometry>
-        <mesh
-          filename="package://robot_description/meshes/right_arm.STL" />
-      </geometry>
-      <material
-        name="">
-        <color
-          rgba="0.75294 0.75294 0.75294 1" />
-      </material>
-    </visual>
-    <collision>
-      <origin
-        xyz="0 0 0"
-        rpy="0 0 0" />
-      <geometry>
-        <mesh
-          filename="package://robot_description/meshes/right_arm.STL" />
-      </geometry>
-    </collision>
-  </link>
-  <joint
-    name="right_arm_fixed"
-    type="fixed">
-    <origin
-      xyz="0 -0.25 0.7"
-      rpy="0 0 0" />
-    <parent
-      link="base_link" />
-    <child
-      link="right_arm" />
-    <axis
-      xyz="0 0 0" />
-  </joint>
-  -->
   <!-- depth camera -->
   <link

Commit message: Pose experiment ready to be run: -Adapted oscar launch and xacro files to allow a fixed load in the grippers -Decreased planing time to 0.05s for arm commands -Created pose_test.launch to set the experiment parameters and launch all nodes -pose_test.py now saves in oscar_test/results folder -pose_test.py sets gazebo unlimits update rate to speedup simulation

File: oscar_description/urdf/oscar.urdf.xacro (robot description, xacro)
@@ -1,202 +1,46 @@
 <?xml version="1.0" encoding="utf-8"?>
-<!-- This URDF was partially created by SolidWorks to URDF Exporter! Originally created by Stephen Brawner (brawner@gmail.com)
-     Commit Version: 1.5.1-0-g916b5db  Build Version: 1.5.7152.31018
-     For more information, please see http://wiki.ros.org/sw_urdf_exporter -->
 <!-- OSCAR: Open Source Cognitive Applied Robot -->
 <!-- Author: Emanuel Fallas -->
 <!-- Lab: LIANA https://www.tec.ac.cr/unidades/laboratorio-inteligencia-artificial-ciencias-naturales-liana -->
-<robot
-  name="oscar" xmlns:xacro="http://ros.org/wiki/xacro">
-  <!-- Import Gazebo plugins -->
-  <xacro:include filename="$(find oscar_description)/urdf/oscar.gazebo"/>
-  <!-- Load Thor robotic arm xacro file -->
-  <xacro:include filename="$(find thor_description)/urdf/thor_description.urdf.xacro"/>
-  <link name="world" />
-  <joint name="base_to_world" type="fixed">
-    <parent link="world"/>
-    <child link="base_link"/>
-  </joint>
-  <link
-    name="base_link">
-    <inertial>
-      <origin
-        xyz="0.0007415 -6.6609E-17 0.53453"
-        rpy="0 0 0" />
-      <mass
-        value="22.41" />
-      <inertia
-        ixx="1.9751"
-        ixy="-6.2222E-17"
-        ixz="-0.0047359"
-        iyy="1.508"
-        iyz="-6.0087E-16"
-        izz="0.62031" />
-    </inertial>
-    <visual>
-      <origin
-        xyz="0 0 0"
-        rpy="0 0 0" />
-      <geometry>
-        <mesh
-          filename="package://oscar_description/meshes/base_link.STL" />
-      </geometry>
-      <material
-        name="">
-        <color
-          rgba="0.79216 0.81961 0.93333 1" />
-      </material>
-    </visual>
-    <collision>
-      <origin
-        xyz="0 0 0"
-        rpy="0 0 0" />
-      <geometry>
-        <mesh
-          filename="package://oscar_description/meshes/base_link.STL" />
-      </geometry>
-    </collision>
-  </link>
-  <!-- Left arm xacro call and joint -->
-  <xacro:thor_robot prefix="left_arm_"/>
-  <joint
-    name="left_arm_fixed"
-    type="fixed">
-    <origin
-      xyz="0 0.25 0.7"
-      rpy="0 0 0" />
-    <parent
-      link="world" />
-    <child
-      link="left_arm_base_link" />
-    <axis
-      xyz="0 0 0" />
-  </joint>
-  <!-- Right arm xacro call and joint -->
-  <xacro:thor_robot prefix="right_arm_"/>
-  <joint
-    name="right_arm_fixed"
-    type="fixed">
-    <origin
-      xyz="0 -0.25 0.7"
-      rpy="0 0 0" />
-    <parent
-      link="world" />
-    <child
-      link="right_arm_base_link" />
-    <axis
-      xyz="0 0 0" />
-  </joint>
-  <!-- depth camera -->
-  <link
-    name="depth_camera_link">
-    <inertial>
-      <origin
-        xyz="-0.013049 0.00024617 -6.059E-05"
-        rpy="0 0 0" />
-      <mass
-        value="0.044752" />
-      <inertia
-        ixx="2.7277E-05"
-        ixy="2.4434E-07"
-        ixz="-1.1786E-09"
-        iyy="3.9447E-06"
-        iyz="-2.818E-09"
-        izz="2.7362E-05" />
-    </inertial>
-    <visual>
-      <origin
-        xyz="0 0 0"
-        rpy="0 0 0" />
-      <geometry>
-        <mesh
-          filename="package://oscar_description/meshes/depth_camera_link.STL" />
-      </geometry>
-      <material
-        name="">
-        <color
-          rgba="0.79216 0.81961 0.93333 1" />
-      </material>
-    </visual>
-    <collision>
-      <origin
-        xyz="0 0 0"
-        rpy="0 0 0" />
-      <geometry>
-        <mesh
-          filename="package://oscar_description/meshes/depth_camera_link.STL" />
-      </geometry>
-    </collision>
-  </link>
-  <joint
-    name="depth_camera_fixed"
-    type="fixed">
-    <origin
-      xyz="0.092973 0 1.703"
-      rpy="0 1.0734 0" />
-    <parent
-      link="base_link" />
-    <child
-      link="depth_camera_link" />
-    <axis
-      xyz="0 0 0" />
-  </joint>
-  <link name="depth_optical_frame" />
-  <joint name="depth_camera_frame_fixed" type="fixed">
-    <parent link="depth_camera_link"/>
-    <child link="depth_optical_frame"/>
-    <origin xyz="0 0 0" rpy="${-pi/2} 0 ${-pi/2}"/>
-  </joint>
-  <link
-    name="rgb_camera_link">
-    <inertial>
-      <origin
-        xyz="-0.0061932 -8.2211E-05 4.4544E-05"
-        rpy="0 0 0" />
-      <mass
-        value="0.0011575" />
-      <inertia
-        ixx="6.7691E-08"
-        ixy="-3.6041E-11"
-        ixz="-2.5249E-13"
-        iyy="3.9729E-08"
-        iyz="1.6534E-13"
-        izz="2.8883E-08" />
-    </inertial>
-    <visual>
-      <origin
-        xyz="0 0 0"
-        rpy="0 0 0" />
-      <geometry>
-        <mesh
-          filename="package://oscar_description/meshes/rgb_camera_link.STL" />
-      </geometry>
-      <material
-        name="">
-        <color
-          rgba="1 1 1 1" />
-      </material>
-    </visual>
-    <collision>
-      <origin
-        xyz="0 0 0"
-        rpy="0 0 0" />
-      <geometry>
-        <mesh
-          filename="package://oscar_description/meshes/rgb_camera_link.STL" />
-      </geometry>
-    </collision>
-  </link>
-  <joint
-    name="rgb_camera_link"
-    type="fixed">
-    <origin
-      xyz="0.42501 0 2.03"
-      rpy="0 1.5708 0" />
-    <parent
-      link="base_link" />
-    <child
-      link="rgb_camera_link" />
-    <axis
-      xyz="0 0 0" />
-  </joint>
+<robot name="oscar" xmlns:xacro="http://ros.org/wiki/xacro">
+  <!-- Import OSCAR xacro -->
+  <xacro:include filename="$(find oscar_description)/urdf/oscar.xacro"/>
+  <xacro:oscar_robot />
+  <xacro:property name="width" value="0.025" />
+  <xacro:arg name="mass" default="0.001" />
+  <xacro:arg name="load" default="false" />
+  <xacro:macro name="generate_box" params="width mass arm" >
+      <link name="load_${arm}">
+      <!--
+      <collision>
+        <origin xyz="0 0 0" rpy="0 0 0"/>
+        <geometry>
+          <box size="${width} ${width} ${width}"/>
+        </geometry>
+      </collision>
+      -->
+      <visual>
+        <origin xyz="0 0 0" rpy="0 0 0"/>
+        <geometry>
+          <box size="${width} ${width} ${width}"/>
+        </geometry>
+      </visual>
+      <inertial>
+        <origin xyz="0 0 0" rpy="0 0 0"/>
+        <mass value="${mass}"/>
+        <inertia
+          ixx="${mass / 12.0 * (width*width + width*width)}" ixy="0.0" ixz="0.0"
+          iyy="${mass / 12.0 * (width*width + width*width)}" iyz="0.0"
+          izz="${mass / 12.0 * (width*width + width*width)}" />
+      </inertial>
+    </link>
+    <joint name="${arm}_load_to_arm" type="fixed">
+        <parent link="${arm}_arm_gripper_link"/>
+        <child link="load_${arm}"/>
+    </joint>
+  </xacro:macro>
+  <xacro:if value="$(arg load)">
+    <xacro:generate_box width="${width}" mass="$(arg mass)" arm="right"/>
+    <xacro:generate_box width="${width}" mass="$(arg mass)" arm="left"/>
+  </xacro:if>
 </robot>

Commit message: Lots of cosmetic and license changes

File: oscar_description/urdf/oscar.urdf.xacro (robot description, xacro)
@@ -1,10 +1,14 @@
 <?xml version="1.0" encoding="utf-8"?>
+<!-- oscar.urdf.xacro: Loads oscar robot and allows to put a fixed load in the arms-->
 <!-- OSCAR: Open Source Cognitive Applied Robot -->
 <!-- Author: Emanuel Fallas -->
-<!-- Lab: LIANA https://www.tec.ac.cr/unidades/laboratorio-inteligencia-artificial-ciencias-naturales-liana -->
+<!-- email: efallashdez@gmail.com -->
+<!-- Published under GNU GPLv3 license -->
 <robot name="oscar" xmlns:xacro="http://ros.org/wiki/xacro">
   <!-- Import OSCAR xacro -->
   <xacro:include filename="$(find oscar_description)/urdf/oscar.xacro"/>
+  <!--Generates oscar robot-->
   <xacro:oscar_robot />
+  <!--Macro to put a fixed load in the arms (used in pose test)-->
   <xacro:property name="width" value="0.025" />
   <xacro:arg name="mass" default="0.001" />
@@ -12,12 +16,4 @@
   <xacro:macro name="generate_box" params="width mass arm" >
       <link name="load_${arm}">
-      <!--
-      <collision>
-        <origin xyz="0 0 0" rpy="0 0 0"/>
-        <geometry>
-          <box size="${width} ${width} ${width}"/>
-        </geometry>
-      </collision>
-      -->
       <visual>
         <origin xyz="0 0 0" rpy="0 0 0"/>
@@ -40,4 +36,5 @@
     </joint>
   </xacro:macro>
+  <!--Calls the fixed load macro-->
   <xacro:if value="$(arg load)">
     <xacro:generate_box width="${width}" mass="$(arg mass)" arm="right"/>

File: oscar_description/urdf/oscar.xacro (robot description, xacro)
@@ -1,16 +1,19 @@
 <?xml version="1.0" encoding="utf-8"?>
+<!-- oscar.xacro: OSCAR Description File-->
+<!-- OSCAR: Open Source Cognitive Applied Robot -->
+<!-- Author: Emanuel Fallas -->
+<!-- email: efallashdez@gmail.com -->
+<!-- Published under GNU GPLv3 license -->
 <!-- This URDF was partially created by SolidWorks to URDF Exporter! Originally created by Stephen Brawner (brawner@gmail.com)
      Commit Version: 1.5.1-0-g916b5db  Build Version: 1.5.7152.31018
      For more information, please see http://wiki.ros.org/sw_urdf_exporter -->
-<!-- OSCAR: Open Source Cognitive Applied Robot -->
-<!-- Author: Emanuel Fallas -->
-<!-- Lab: LIANA https://www.tec.ac.cr/unidades/laboratorio-inteligencia-artificial-ciencias-naturales-liana -->
 <robot xmlns:xacro="http://ros.org/wiki/xacro">
   <!-- MAIN MACRO: Generates the URDF of the OSCAR Robot-->
   <xacro:macro name="oscar_robot" >
-    <!-- Import Gazebo plugins -->
+    <!--Imports Gazebo plugins-->
     <xacro:include filename="$(find oscar_description)/urdf/oscar.gazebo"/>
-    <!-- Load Thor robotic arm xacro file -->
+    <!--Loads Thor robotic arm xacro file-->
     <xacro:include filename="$(find thor_description)/urdf/thor_description.urdf.xacro"/>
+    <!--World gazebo frame-->
     <link name="world" />
     <joint name="base_to_world" type="fixed">
@@ -142,4 +145,5 @@
         xyz="0 0 0" />
     </joint>
+    <!--Optical frame to orient the point cloud properly-->
     <link name="depth_optical_frame" />
     <joint name="depth_camera_frame_fixed" type="fixed">
@@ -148,4 +152,5 @@
       <origin xyz="0 0 0" rpy="${-pi/2} 0 ${-pi/2}"/>
     </joint>
+    <!--RGB camera-->
     <link
       name="rgb_camera_link">
